File: LCD_Back_Neo_Key_RxTx_emergency_stop/drill_holes.sch (KiCad schematic (older format))
At the start: 2 parts, among them J4 Display_support_pin, J5 Display_support_pin

Commit message: update
Parts:
- J4, J5: symbol Connector:Conn_01x01_Female -> LCD_Back_Neo_Key_RxTx_emergency_stop-rescue:Conn_01x01_Female-Connector
Changed lines of the file:
@@
 $EndDescr
 $Comp
-L Connector:Conn_01x01_Female J?
+L LCD_Back_Neo_Key_RxTx_emergency_stop-rescue:Conn_01x01_Female-Connector J?
 U 1 1 5CF1CF44
 P 1150 950
@@
 $EndComp
 $Comp
-L Connector:Conn_01x01_Female J?
+L LCD_Back_Neo_Key_RxTx_emergency_stop-rescue:Conn_01x01_Female-Connector J?
 U 1 1 5CF1CF4A
 P 1150 1250
