File: LCD_Back_Neo_Key_RxTx_emergency_stop/display.sch (KiCad schematic (older format))
At the start: 5 parts, among them J2 Conn_01x20_Female, Q1 BC337

Commit message: update
Parts:
- C1: symbol Device:CP -> LCD_Back_Neo_Key_RxTx_emergency_stop-rescue:CP-Device
- Q1: symbol Transistor_BJT:BC337 -> LCD_Back_Neo_Key_RxTx_emergency_stop-rescue:BC337-Transistor_BJT
- R1, R2: symbol Device:R -> LCD_Back_Neo_Key_RxTx_emergency_stop-rescue:R-Device
Changed lines of the file:
@@
 VCC-5V
 $Comp
-L Device:CP C?
+L LCD_Back_Neo_Key_RxTx_emergency_stop-rescue:CP-Device C?
 U 1 1 5CEEE166
 P 6650 4450
@@
 $EndComp
 $Comp
-L Device:R R?
+L LCD_Back_Neo_Key_RxTx_emergency_stop-rescue:R-Device R?
 U 1 1 5CEEE16C
 P 6300 4300
@@
 	5950 4300 6150 4300
 $Comp
-L Transistor_BJT:BC337 Q?
+L LCD_Back_Neo_Key_RxTx_emergency_stop-rescue:BC337-Transistor_BJT Q?
 U 1 1 5CEEE177
 P 4850 4300
@@
 $EndComp
 $Comp
-L Device:R R?
+L LCD_Back_Neo_Key_RxTx_emergency_stop-rescue:R-Device R?
 U 1 1 5CEEE17D
 P 4250 4300

Commit message: move keyboard connector
Parts:
- R2: footprint Resistor_THT:R_Axial_DIN0207_L6.3mm_D2.5mm_P15.24mm_Horizontal -> Resistor_THT:R_Axial_DIN0207_L6.3mm_D2.5mm_P10.16mm_Horizontal
Changed lines of the file:
@@
 F 0 "R2" V 6093 4300 50  0000 C CNN
 F 1 "R" V 6184 4300 50  0000 C CNN
-F 2 "Resistor_THT:R_Axial_DIN0207_L6.3mm_D2.5mm_P15.24mm_Horizontal" V 6185 4300 50  0001 C CNN
+F 2 "Resistor_THT:R_Axial_DIN0207_L6.3mm_D2.5mm_P10.16mm_Horizontal" V 6185 4300 50  0001 C CNN
 F 3 "~" H 6300 4300 50  0001 C CNN
 	1    6300 4300
